File: can.sch (KiCad schematic (older format))
At the start: 13 parts, among them P7 CAN, U10 MCP2551-I/SN, U11 MCP2515, U12 SG-210STF_16MHz

Commit message: Fixed MCP2525 wrong package
Signed-off-by: Akira Tsukamoto <akira-t@s9.dion.ne.jp>
Parts:
- U11: symbol MCP2515 -> MCP2515-TSSOP20
Connections:
- net +3V3: now also U11.20 (Vdd); no longer U11.18 (Vdd)
- net GND: now also U11.10 (Vss_GND); no longer U11.9 (Vss_GND)
- net MISO: now also U11.17 (SO); no longer U11.15 (SO)
- net MOSI: now also U11.16 (SI); no longer U11.14 (SI)
- net SCLK: now also U11.14 (SCK); no longer U11.13 (SCK)
- net ~CAN_CS: now also U11.18 (~CS); no longer U11.16 (~CS)
- net ~CAN_IRQ: now also U11.13 (~INT); no longer U11.12 (~INT)
- net ~RESET: now also U11.19 (~RESET); no longer U11.17 (~RESET)
- net at TH15.1, U12.3 (OUT): now also U11.9 (OSC1); no longer U11.8 (OSC1)
Changed lines of the file:
@@
 Title "DCoJA Yatagarasu Mezzanine"
 Date "2017-03-31"
-Rev "0.10"
+Rev "0.10.1"
 Comp "DroneWorks Inc."
 Comment1 "Copyright (c) 2017 DroneWorks Inc."
@@
 $EndDescr
 $Comp
-L MCP2515 U11
+L MCP2515-TSSOP20 U11
 U 1 1 56F7C46B
 P 4600 3850
